File: eagle/dci.sch (EAGLE design)
At the start: 87 parts, among them IC1 7406N, IC10 4029N, IC11 4029N, IC12 4081N, IC2 4013N, IC3 4013N, IC4 4029N, IC5 4029N, IC6 4081N, IC7 7406N, IC8 4013N, IC9 4013N, J1 455-1750-1-ND, J10 455-1750-1-ND, J11 455-1750-1-ND, J12 455-1750-1-ND, J13 455-1750-1-ND, J14 455-1750-1-ND, J2 455-1750-1-ND, J3 455-1750-1-ND, J4 455-1750-1-ND, J5 455-1750-1-ND

Commit message: Organize the DCI schematic
Connections:
- net 1200_EN renamed /1200_EN
- net 300_EN renamed /300_EN
- net 600_EN renamed /600_EN
- net LOW_1 renamed LOW_WRITE_1
- net LOW_3 renamed LOW_READ_1
- net SERV_REQ renamed /SERV_REQ
- net ~1200_EN renamed ~/1200_EN
- net ~300_EN renamed ~/300_EN
Other:
- moved on the sheet: U$24, U$25G$5
Changed lines of the file:
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@@
 <instance part="IC10" gate="A" x="281.94" y="109.22"/>
 <instance part="IC11" gate="A" x="226.06" y="106.68"/>
-<instance part="U$24" gate="G$1" x="248.92" y="195.58"/>
+<instance part="U$24" gate="G$1" x="254" y="195.58"/>
 <instance part="U$25" gate="G$1" x="424.18" y="106.68"/>
 <instance part="U$25" gate="G$2" x="424.18" y="88.9"/>
 <instance part="U$25" gate="G$4" x="474.98" y="88.9"/>
-<instance part="U$25" gate="G$5" x="213.36" y="187.96"/>
+<instance part="U$25" gate="G$5" x="218.44" y="187.96"/>
 <instance part="U$25" gate="G$6" x="474.98" y="106.68"/>
 <instance part="RN1" gate="G$1" x="147.32" y="279.4"/>
@@
 <instance part="P+25" gate="VCC" x="210.82" y="121.92"/>
 <instance part="GND40" gate="1" x="208.28" y="88.9"/>
-<instance part="GND41" gate="1" x="233.68" y="180.34"/>
+<instance part="GND41" gate="1" x="238.76" y="180.34"/>
 <instance part="GND43" gate="1" x="452.12" y="330.2"/>
 <instance part="P+26" gate="VCC" x="139.7" y="292.1"/>
@@
 <segment>
 <pinref part="U$24" gate="G$1" pin="1A"/>
-<wire x1="236.22" y1="205.74" x2="233.68" y2="205.74" width="0.1524" layer="91"/>
-<wire x1="233.68" y1="205.74" x2="233.68" y2="203.2" width="0.1524" layer="91"/>
+<wire x1="241.3" y1="205.74" x2="238.76" y2="205.74" width="0.1524" layer="91"/>
+<wire x1="238.76" y1="205.74" x2="238.76" y2="203.2" width="0.1524" layer="91"/>
 <pinref part="U$24" gate="G$1" pin="2A"/>
-<wire x1="233.68" y1="203.2" x2="236.22" y2="203.2" width="0.1524" layer="91"/>
-<wire x1="233.68" y1="203.2" x2="233.68" y2="185.42" width="0.1524" layer="91"/>
-<junction x="233.68" y="203.2"/>
+<wire x1="238.76" y1="203.2" x2="241.3" y2="203.2" width="0.1524" layer="91"/>
+<wire x1="238.76" y1="203.2" x2="238.76" y2="185.42" width="0.1524" layer="91"/>
+<junction x="238.76" y="203.2"/>
 <pinref part="U$24" gate="G$1" pin="DIS2"/>
-<wire x1="233.68" y1="185.42" x2="236.22" y2="185.42" width="0.1524" layer="91"/>
-<wire x1="233.68" y1="185.42" x2="233.68" y2="182.88" width="0.1524" layer="91"/>
-<junction x="233.68" y="185.42"/>
+<wire x1="238.76" y1="185.42" x2="241.3" y2="185.42" width="0.1524" layer="91"/>
+<wire x1="238.76" y1="185.42" x2="238.76" y2="182.88" width="0.1524" layer="91"/>
+<junction x="238.76" y="185.42"/>
 <pinref part="GND41" gate="1" pin="GND"/>
 </segment>
@@
 </segment>
 </net>
-<net name="LOW_1" class="0">
-<segment>
-<wire x1="287.02" y1="182.88" x2="294.64" y2="182.88" width="0.1524" layer="91"/>
+<net name="LOW_WRITE_1" class="0">
+<segment>
+<wire x1="276.86" y1="182.88" x2="294.64" y2="182.88" width="0.1524" layer="91"/>
 <pinref part="IC12" gate="B" pin="I1"/>
-<label x="287.02" y="182.88" size="1.778" layer="95"/>
+<label x="276.86" y="182.88" size="1.778" layer="95"/>
 </segment>
 <segment>
 <pinref part="IC12" gate="A" pin="I1"/>
-<wire x1="294.64" y1="170.18" x2="287.02" y2="170.18" width="0.1524" layer="91"/>
-<label x="287.02" y="170.18" size="1.778" layer="95"/>
+<wire x1="294.64" y1="170.18" x2="276.86" y2="170.18" width="0.1524" layer="91"/>
+<label x="276.86" y="170.18" size="1.778" layer="95"/>
 </segment>
 <segment>
@@
 <segment>
 <pinref part="U$24" gate="G$1" pin="6Y"/>
-<wire x1="261.62" y1="193.04" x2="266.7" y2="193.04" width="0.1524" layer="91"/>
-<label x="264.16" y="193.04" size="1.778" layer="95"/>
+<wire x1="266.7" y1="193.04" x2="271.78" y2="193.04" width="0.1524" layer="91"/>
+<label x="269.24" y="193.04" size="1.778" layer="95"/>
 </segment>
 <segment>
@@
 <segment>
 <pinref part="U$24" gate="G$1" pin="5Y"/>
-<wire x1="261.62" y1="195.58" x2="266.7" y2="195.58" width="0.1524" layer="91"/>
-<label x="264.16" y="195.58" size="1.778" layer="95"/>
+<wire x1="266.7" y1="195.58" x2="271.78" y2="195.58" width="0.1524" layer="91"/>
+<label x="269.24" y="195.58" size="1.778" layer="95"/>
 </segment>
 <segment>
@@
 </segment>
 </net>
-<net name="300_EN" class="0">
+<net name="/300_EN" class="0">
 <segment>
 <wire x1="454.66" y1="106.68" x2="464.82" y2="106.68" width="0.1524" layer="91"/>
@@
 </segment>
 </net>
-<net name="600_EN" class="0">
+<net name="/600_EN" class="0">
 <segment>
 <pinref part="RN6" gate="G" pin="1"/>
@@
 <segment>
 <pinref part="U$24" gate="G$1" pin="4A"/>
-<wire x1="236.22" y1="198.12" x2="220.98" y2="198.12" width="0.1524" layer="91"/>
-<label x="220.98" y="198.12" size="1.778" layer="95"/>
+<wire x1="241.3" y1="198.12" x2="226.06" y2="198.12" width="0.1524" layer="91"/>
+<label x="226.06" y="198.12" size="1.778" layer="95"/>
 </segment>
 <segment>
@@
 <segment>
 <pinref part="U$24" gate="G$1" pin="6A"/>
-<wire x1="220.98" y1="193.04" x2="236.22" y2="193.04" width="0.1524" layer="91"/>
-<label x="220.98" y="193.04" size="1.778" layer="95"/>
+<wire x1="226.06" y1="193.04" x2="241.3" y2="193.04" width="0.1524" layer="91"/>
+<label x="226.06" y="193.04" size="1.778" layer="95"/>
 </segment>
 <segment>
@@
 <segment>
 <pinref part="U$24" gate="G$1" pin="5A"/>
-<wire x1="236.22" y1="195.58" x2="220.98" y2="195.58" width="0.1524" layer="91"/>
-<label x="220.98" y="195.58" size="1.778" layer="95"/>
+<wire x1="241.3" y1="195.58" x2="226.06" y2="195.58" width="0.1524" layer="91"/>
+<label x="226.06" y="195.58" size="1.778" layer="95"/>
 </segment>
 </net>
@@
 <segment>
 <pinref part="U$24" gate="G$1" pin="DIS1"/>
-<wire x1="236.22" y1="187.96" x2="223.52" y2="187.96" width="0.1524" layer="91"/>
+<wire x1="241.3" y1="187.96" x2="228.6" y2="187.96" width="0.1524" layer="91"/>
 <pinref part="U$25" gate="G$5" pin="Z"/>
 </segment>
@@
 <segment>
 <pinref part="U$24" gate="G$1" pin="3Y"/>
-<wire x1="261.62" y1="200.66" x2="266.7" y2="200.66" width="0.1524" layer="91"/>
-<label x="264.16" y="200.66" size="1.778" layer="95"/>
+<wire x1="266.7" y1="200.66" x2="271.78" y2="200.66" width="0.1524" layer="91"/>
+<label x="269.24" y="200.66" size="1.778" layer="95"/>
 </segment>
 <segment>
@@
 <segment>
 <pinref part="U$24" gate="G$1" pin="4Y"/>
-<wire x1="261.62" y1="198.12" x2="266.7" y2="198.12" width="0.1524" layer="91"/>
-<label x="264.16" y="198.12" size="1.778" layer="95"/>
+<wire x1="266.7" y1="198.12" x2="271.78" y2="198.12" width="0.1524" layer="91"/>
+<label x="269.24" y="198.12" size="1.778" layer="95"/>
 </segment>
 <segment>
@@
 </segment>
 </net>
-<net name="LOW_3" class="0">
+<net name="LOW_READ_1" class="0">
 <segment>
 <pinref part="U$25" gate="G$5" pin="A"/>
-<wire x1="203.2" y1="187.96" x2="193.04" y2="187.96" width="0.1524" layer="91"/>
-<label x="193.04" y="187.96" size="1.778" layer="95"/>
+<wire x1="208.28" y1="187.96" x2="190.5" y2="187.96" width="0.1524" layer="91"/>
+<label x="190.5" y="187.96" size="1.778" layer="95"/>
 </segment>
 <segment>
@@
 </segment>
 </net>
-<net name="SERV_REQ" class="0">
+<net name="/SERV_REQ" class="0">
 <segment>
 <pinref part="R6" gate="G$1" pin="2"/>
@@
 </segment>
 </net>
-<net name="1200_EN" class="0">
+<net name="/1200_EN" class="0">
 <segment>
 <pinref part="IC11" gate="A" pin="J3"/>
@@
 </segment>
 </net>
-<net name="~300_EN" class="0">
+<net name="~/300_EN" class="0">
 <segment>
 <pinref part="IC11" gate="A" pin="J4"/>
@@
 </segment>
 </net>
-<net name="~1200_EN" class="0">
+<net name="~/1200_EN" class="0">
 <segment>
 <pinref part="U$25" gate="G$4" pin="Z"/>
@@
 <segment>
 <pinref part="U$24" gate="G$1" pin="3A"/>
-<wire x1="220.98" y1="200.66" x2="236.22" y2="200.66" width="0.1524" layer="91"/>
-<label x="220.98" y="200.66" size="1.778" layer="95"/>
-</segment>
-</net>
+<wire x1="226.06" y1="200.66" x2="241.3" y2="200.66" width="0.1524" layer="91"/>
+<label x="226.06" y="200.66" size="1.778" layer="95"/>
+</segment>
+</net>
