File: eagle/processor.sch (EAGLE design)
At the start: 106 parts, among them IC1 74LS145N, IC10 74LS74N, IC13 74LS92N, IC14 74LS06N, IC15 7407N, IC16 74LS04N, IC17 74LS191N, IC18 74LS14N, IC19 74S74N, IC2 74LS145N, IC20 74S03N, IC21 74LS20N, IC22 74LS74N, IC23 74LS00N, IC24 74LS145N, IC25 74LS145N, IC26 74LS00N, IC27 74LS02N, IC28 4049N, IC29 74LS279N, IC3 74LS00N, IC30 74154N, IC31 74LS293N, IC32 4050N, IC33 74LS74N, IC34 ROM1, IC35 ROM0, IC36 74LS92N, IC37 74LS06N, IC38 7407N, IC39 74LS04N, IC4 74LS02N, IC40 74LS191N, IC41 74LS14N, IC42 74S74N, IC43 74S03N, IC44 74LS20N, IC45 74LS74N, IC46 74LS00N, IC5 4049N, IC6 74LS279N, IC7 74154N, IC8 74LS293N, IC9 4050N, Q1 2N3906, Q10 2N3904, Q2 2N3906, Q3 2N3906, Q4 2N3906, Q5 2N3906, Q6 2N3906, Q7 2N3904, Q8 2N3904, Q9 2N3904

Commit message: Organize the DCI schematic
Connections:
- net LOW_0 renamed WRITE_0
- net LOW_1 renamed WRITE_1
- net LOW_2 renamed READ_0
- net LOW_3 renamed READ_1
- net MC5.6 renamed /INT
- net ~IC33B renamed /SERV_REQ
- net ~J1_CLK renamed ~/J1_CLK
- new net LOW_READ_0: JP8.58.1, U$22.3Y
- new net LOW_READ_1: JP8.60.1, U$22.2Y
- new net LOW_WRITE_0: JP8.62.1, U$22.4Y
- new net LOW_WRITE_1: JP8.64.1, U$22.1Y
- net J1.58: no longer JP8.58.1, U$22.3Y
- net J1.60: no longer JP8.60.1, U$22.2Y
- net J1.62: no longer JP8.62.1, U$22.4Y
- net J1.64: no longer JP8.64.1, U$22.1Y
Changed lines of the file:
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@@
 </segment>
 </net>
-<net name="J1.58" class="0">
+<net name="LOW_READ_0" class="0">
 <segment>
 <pinref part="JP8" gate=".58" pin="1"/>
@@
 </segment>
 </net>
-<net name="J1.60" class="0">
+<net name="LOW_READ_1" class="0">
 <segment>
 <pinref part="U$22" gate="G$1" pin="2Y"/>
@@
 </segment>
 </net>
-<net name="J1.62" class="0">
+<net name="LOW_WRITE_0" class="0">
 <segment>
 <pinref part="U$22" gate="G$1" pin="4Y"/>
@@
 </segment>
 </net>
-<net name="J1.64" class="0">
+<net name="LOW_WRITE_1" class="0">
 <segment>
 <pinref part="U$22" gate="G$1" pin="1Y"/>
@@
 </segment>
 </net>
-<net name="~IC33B" class="0">
+<net name="/SERV_REQ" class="0">
 <segment>
 <pinref part="JP8" gate=".66" pin="1"/>
@@
 </segment>
 <segment>
-<wire x1="215.9" y1="398.78" x2="205.74" y2="398.78" width="0.1524" layer="91"/>
-<label x="205.74" y="398.78" size="1.778" layer="95"/>
+<wire x1="215.9" y1="398.78" x2="200.66" y2="398.78" width="0.1524" layer="91"/>
+<label x="200.66" y="398.78" size="1.778" layer="95"/>
 <pinref part="Q7" gate="G1" pin="B"/>
 </segment>
@@
 <segment>
 <pinref part="IC44" gate="A" pin="I1"/>
-<wire x1="594.36" y1="330.2" x2="589.28" y2="330.2" width="0.1524" layer="91"/>
-<label x="589.28" y="330.2" size="1.778" layer="95"/>
+<wire x1="594.36" y1="330.2" x2="579.12" y2="330.2" width="0.1524" layer="91"/>
+<label x="579.12" y="330.2" size="1.778" layer="95"/>
 </segment>
 </net>
@@
 <segment>
 <pinref part="IC46" gate="D" pin="I0"/>
-<wire x1="543.56" y1="325.12" x2="538.48" y2="325.12" width="0.1524" layer="91"/>
-<label x="538.48" y="325.12" size="1.778" layer="95"/>
+<wire x1="543.56" y1="325.12" x2="535.94" y2="325.12" width="0.1524" layer="91"/>
+<label x="535.94" y="325.12" size="1.778" layer="95"/>
 </segment>
 <segment>
@@
 </segment>
 </net>
-<net name="LOW_0" class="0">
+<net name="WRITE_0" class="0">
 <segment>
 <pinref part="U$22" gate="G$1" pin="4A"/>
@@
 </segment>
 </net>
-<net name="LOW_1" class="0">
+<net name="WRITE_1" class="0">
 <segment>
 <pinref part="U$18" gate="G$1" pin="Q2"/>
@@
 </segment>
 </net>
-<net name="LOW_3" class="0">
+<net name="READ_1" class="0">
 <segment>
 <pinref part="U$18" gate="G$1" pin="Q4"/>
@@
 </segment>
 </net>
-<net name="~J1_CLK" class="0">
+<net name="~/J1_CLK" class="0">
 <segment>
 <pinref part="IC45" gate="B" pin="CLK"/>
@@
 </segment>
 </net>
-<net name="MC5.6" class="0">
+<net name="/INT" class="0">
 <segment>
 <pinref part="IC46" gate="C" pin="O"/>
@@
 </segment>
 </net>
-<net name="LOW_2" class="0">
+<net name="READ_0" class="0">
 <segment>
 <pinref part="U$18" gate="G$1" pin="Q3"/>
